Commit message: Completed Lab 7

File: lab7/urdf/rtr_manipulator.xacro (robot description, xacro)
@@ -1,5 +1,4 @@
 <?xml version="1.0"?>
 <robot xmlns:xacro="http://www.ros.org/wiki/xacro" name="rtr_manipulator">
-  <!-- RTR: Revolute (base yaw) – Prismatic (vertical) – Revolute (elbow). -->
   <xacro:property name="l2" value="0.9"/>
   <xacro:property name="l3" value="1.0"/>
@@ -10,5 +9,4 @@
   <material name="grey"><color rgba="0.7 0.7 0.7 1"/></material>
   <link name="world"/>
-  <!-- Origins chosen so joint variables match the paper FK (no extra vertical offset in theta_2). -->
   <link name="base_link">
     <visual>
@@ -17,4 +15,8 @@
       <material name="grey"/>
     </visual>
+    <collision>
+      <origin xyz="0 0 0.05" rpy="0 0 0"/>
+      <geometry><cylinder radius="0.12" length="0.1"/></geometry>
+    </collision>
   </link>
   <joint name="world_to_base" type="fixed">
@@ -34,4 +36,8 @@
       <material name="blue"/>
     </visual>
+    <collision>
+      <origin xyz="0 0 0.15" rpy="0 0 0"/>
+      <geometry><cylinder radius="0.06" length="0.3"/></geometry>
+    </collision>
   </link>
   <joint name="joint_theta1" type="revolute">
@@ -53,4 +59,8 @@
       <material name="green"/>
     </visual>
+    <collision>
+      <origin xyz="0 0 0" rpy="0 0 0"/>
+      <geometry><box size="${width} ${width} ${width}"/></geometry>
+    </collision>
   </link>
   <joint name="joint_theta2" type="prismatic">
@@ -72,4 +82,8 @@
       <material name="red"/>
     </visual>
+    <collision>
+      <origin xyz="${l2/2} 0 0" rpy="0 0 0"/>
+      <geometry><box size="${l2} ${width} ${width}"/></geometry>
+    </collision>
   </link>
   <joint name="fixed_carriage_upper" type="fixed">
@@ -89,4 +103,8 @@
       <material name="blue"/>
     </visual>
+    <collision>
+      <origin xyz="${l3/2} 0 0" rpy="0 0 0"/>
+      <geometry><box size="${l3} ${width} ${width}"/></geometry>
+    </collision>
   </link>
   <joint name="joint_theta3" type="revolute">
@@ -103,5 +121,4 @@
     <origin xyz="${l3} 0 0" rpy="0 0 0"/>
   </joint>
-  <!-- Ignored by joint_state_publisher_gui / classic chain; required for ros2_control bringup. -->
   <ros2_control name="RTRMock" type="system">
     <hardware>
